Commit message: TODO: fix sky texture bug

File: urdf/agriculture_geometry.urdf.xacro (robot description, xacro)
@@ -2,5 +2,5 @@
 <robot name="agriculture_world" xmlns:xacro="http://www.ros.org/wiki/xacro">
   <xacro:property name="package_path" value="$(find arm_mazzolini)"/>
-  <xacro:property name="mesh_path" value="${package_path}/meshes/argiculture_world"/>
+  <xacro:property name="mesh_path" value="${package_path}/meshes/agriculture_world"/>
   <link name="agriculture_world_link">
     <inertial>

File: urdf/base_station.urdf.xacro (robot description, xacro)
@@ -2,5 +2,5 @@
 <robot xmlns:xacro="http://wiki.ros.org/xacro" name="clearpath_base_station">
   <xacro:property name="package_path" value="$(find arm_mazzolini)"/>
-  <xacro:property name="mesh_path" value="${package_path}/meshes/argiculture_world"/>
+  <xacro:property name="mesh_path" value="${package_path}/meshes/agriculture_world"/>
   <xacro:macro name="cpr_base_station" params="name parent *origin">
     <link name="${name}_link">

File: urdf/charge_dock.urdf.xacro (robot description, xacro)
@@ -3,5 +3,5 @@
   <xacro:macro name="cpr_charge_dock" params="name parent *origin">
   <xacro:property name="package_path" value="$(find arm_mazzolini)"/>
-  <xacro:property name="mesh_path" value="${package_path}/meshes/argiculture_world"/>
+  <xacro:property name="mesh_path" value="${package_path}/meshes/agriculture_world"/>
     <link name="${name}_link">
       <visual>
