Commit message: completed image pipeline

File: urdf/camera.xacro (robot description, xacro)
@@ -8,5 +8,6 @@
     <xacro:property name="fps" value="30" />
     <xacro:property name="hfov" value="${PI/3}" />
-    <xacro:property name="name_prefix" value="/camera" />
+    <xacro:property name="name_prefix" value="/simulated_D435" />
+    <!-- TODO: This file is valid only in simulation, change use_sim_time if condition -->
     <xacro:macro name="depth_camera" params= "is_light use_sim_time">
         <link name="camera_link">
@@ -68,8 +69,8 @@
                 <lens>
                     <intrinsics>
-                    <fx>277.1</fx>
-                    <fy>277.1</fy>
-                    <cx>160.5</cx>
-                    <cy>120.5</cy>
+                    <fx>1108.4</fx>
+                    <fy>831.3</fy>
+                    <cx>640</cx>
+                    <cy>360</cy>
                     <s>0</s>
                     </intrinsics>
@@ -90,22 +91,22 @@
                 <clip>
                     <near>0.01</near>
-                    <far>30</far>
+                    <far>30.0</far>
                 </clip>
                 <depth_camera>
                     <clip>
                     <near>0.1</near>
-                    <far>10</far>
+                    <far>10.0</far>
                     </clip>
                 </depth_camera>
                 <noise>
                     <type>gaussian</type>
-                    <mean>0</mean>
+                    <mean>0.0</mean>
                     <stddev>0.003</stddev>
                 </noise>
                 </camera>
                 <always_on>1</always_on>
-                <update_rate>10</update_rate>
+                <update_rate>30</update_rate>
                 <visualize>0</visualize>
-                <topic>/camera/d435/image_raw</topic>
+                <topic>${name_prefix}</topic>
             </sensor>
         </gazebo>

Commit message: visual servoing work in progress

File: urdf/camera.xacro (robot description, xacro)
@@ -44,5 +44,5 @@
             </xacro:if>
             <child link="camera_link"/>
-            <origin xyz="${l2/3} 0 ${-h2-0.03}" rpy="${PI+PI/9} 0 ${-PI/2}"/>
+            <origin xyz="${l2/3} 0 ${-h2-0.03}" rpy="${PI+PI/18} 0 ${-PI/2}"/>
         </joint>
         <link name="camera_kinematic"/>

File: urdf/weeder_robot.xacro (robot description, xacro)
@@ -58,5 +58,5 @@
                 <publish_model_pose>true</publish_model_pose>
                 <publish_link_pose>false</publish_link_pose>
-                <update_frequency>50</update_frequency>
+                <update_frequency>20</update_frequency>
             </plugin>
         </gazebo>
