Commit message: camera work in progress

File: urdf/arm.xacro (robot description, xacro)
@@ -115,4 +115,15 @@
             </link>
         </xacro:if>
+        <link name="camera_link"></link>
+        <joint name="camera_joint" type="fixed">
+            <xacro:unless value="${is_light}">
+                <parent link="link2_heavy"/>
+            </xacro:unless>
+            <xacro:if value="${is_light}">
+                <parent link="link2_light"/>
+            </xacro:if>
+            <child link="camera_link"/>
+            <origin xyz="${l2/2} 0 ${-0.05}" rpy="${PI} 0 ${-PI/2}"/>
+        </joint>
         <!-- Joint 1 (Revolute) -->
         <joint name="joint1" type="revolute">
@@ -122,5 +133,5 @@
             <!-- <origin xyz="0 0 ${h0}" rpy="0 0 0"/> -->
             <axis xyz="0 0 1"/>
-            <limit effort="10" lower="-${PI}" upper="${PI}" velocity="1000"/>
+            <limit effort="100" lower="-${PI}" upper="${PI}" velocity="1000"/>
         </joint>
         <!-- Joint 2 (Revolute) -->
@@ -135,5 +146,5 @@
             <origin xyz="${l1} 0 ${h1}" rpy="0 0 0"/>
             <axis xyz="0 0 1"/>
-            <limit effort="10" lower="-${PI}" upper="${PI}" velocity="1000"/>
+            <limit effort="100" lower="-${PI}" upper="${PI}" velocity="1000"/>
         </joint>
     </xacro:macro>

File: urdf/weeder_robot.xacro (robot description, xacro)
@@ -3,23 +3,13 @@
     <xacro:property name="PI" value="3.141592" />
     <!-- Parameters  -->
-    <xacro:arg name= "is_wheeled" default="false"/>
     <xacro:arg name= "is_light" default="true"/>
+    <xacro:arg name="use_camera" default="true"/>
     <xacro:arg name= "controller_yaml" default=""/>
-    <xacro:macro name="weeder_robot" params="is_wheeled is_light controller_yaml">
+    <xacro:macro name="weeder_robot" params="is_light use_camera controller_yaml">
         <!-- Including base and arm xacro files -->
-        <xacro:unless value="${is_wheeled}">
-            <xacro:include filename="$(find arm_mazzolini)/urdf/base.xacro"/>
-        </xacro:unless>
-        <xacro:if value="${is_wheeled}">
-            <xacro:include filename="$(find arm_mazzolini)/urdf/bunker_fake.xacro"/>
-        </xacro:if>
+        <xacro:include filename="$(find arm_mazzolini)/urdf/bunker_fake.xacro"/>
         <xacro:include filename="$(find arm_mazzolini)/urdf/arm.xacro"/>
         <!-- Create base -->
-        <xacro:unless value="${is_wheeled}">
-            <xacro:base/>
-        </xacro:unless>
-        <xacro:if value="${is_wheeled}">
-            <xacro:bunker_fake/>
-        </xacro:if>
+        <xacro:bunker_fake/>
         <!-- Create robotic arm -->
         <xacro:arm is_light="${is_light}"/>
@@ -27,10 +17,5 @@
         <!-- Fixed joint connecting base_link and arm_base_link -->
         <joint name="base_to_arm_joint" type="fixed">
-            <xacro:unless value="${is_wheeled}">
-                <parent link="base_box"/>
-            </xacro:unless>
-            <xacro:if value="${is_wheeled}">
-                <parent link="base_link"/>
-            </xacro:if>
+            <parent link="base_link"/>
             <child link="arm_base_link"/>
             <origin xyz="0 -0.3 0.28" rpy="0 0 -${PI/2}"/>
@@ -43,10 +28,8 @@
             <xacro:joint_control name="joint1"/>
             <xacro:joint_control name="joint2"/>
-            <xacro:if value="${is_wheeled}">
-                <xacro:wheel_control name="front_left_wheel"/>
-                <xacro:wheel_control name="rear_left_wheel"/>
-                <xacro:wheel_control name="front_right_wheel"/>
-                <xacro:wheel_control name="rear_right_wheel"/>
-            </xacro:if>
+            <xacro:wheel_control name="front_left_wheel"/>
+            <xacro:wheel_control name="rear_left_wheel"/>
+            <xacro:wheel_control name="front_right_wheel"/>
+            <xacro:wheel_control name="rear_right_wheel"/>
         </ros2_control>
         <!-- Gazebo Plugins -->
@@ -64,5 +47,10 @@
             </sensor> -->
         </gazebo>
+        <!-- Add camera simulation -->
+        <xacro:if value="${use_camera}">
+            <xacro:include filename="$(find arm_mazzolini)/urdf/stereo_camera.sdf.xacro"/>
+            <xacro:stereo_camera/>
+        </xacro:if>
     </xacro:macro>
-    <xacro:weeder_robot is_wheeled="$(arg is_wheeled)" is_light="$(arg is_light)" controller_yaml="$(arg controller_yaml)"/>
+    <xacro:weeder_robot is_light="$(arg is_light)" controller_yaml="$(arg controller_yaml)"/>
 </robot>

Commit message: work in progress stereo camera

File: urdf/arm.xacro (robot description, xacro)
@@ -7,12 +7,13 @@
     <xacro:property name="link2_heavy_mesh" value="file://$(find arm_mazzolini)/meshes/stl/Braccio2.stl"/>
     <xacro:property name="link2_light_mesh" value="file://$(find arm_mazzolini)/meshes/stl/Braccio3.stl"/>
+    <xacro:property name="camera_mesh" value="file://$(find arm_mazzolini)/meshes/stl/D435.stl"/>
     <xacro:property name="h0" value="0.07"/>
     <xacro:property name="l0" value="0.190"/>
     <xacro:property name="h1" value="0.0"/>
     <xacro:property name="l1" value="0.190"/>
-    <xacro:property name="h2" value="-0.034"/>
+    <xacro:property name="h2" value="-0.037"/>
     <xacro:property name="l2" value="0.250"/>
     <xacro:property name="scale" value="1e-3 1e-3 1e-3"/>
-    <xacro:macro name="arm" params= "is_light">
+    <xacro:macro name="arm" params= "is_light use_camera">
         <!-- Base Link of robotic arm-->
         <link name="arm_base_link">
@@ -115,15 +116,28 @@
             </link>
         </xacro:if>
-        <link name="camera_link"></link>
-        <joint name="camera_joint" type="fixed">
-            <xacro:unless value="${is_light}">
-                <parent link="link2_heavy"/>
-            </xacro:unless>
-            <xacro:if value="${is_light}">
-                <parent link="link2_light"/>
-            </xacro:if>
-            <child link="camera_link"/>
-            <origin xyz="${l2/2} 0 ${-0.05}" rpy="${PI} 0 ${-PI/2}"/>
-        </joint>
+        <xacro:if value="${use_camera}">
+            <link name="camera_link">
+                <visual>
+                    <geometry>
+                        <mesh filename="${camera_mesh}" scale="${scale}*1000"/>
+                    </geometry>
+                </visual>
+                <collision>
+                    <geometry>
+                        <mesh filename="${camera_mesh}" scale="${scale}*1000"/>
+                    </geometry>
+                </collision>
+            </link>
+            <joint name="camera_joint" type="fixed">
+                <xacro:unless value="${is_light}">
+                    <parent link="link2_heavy"/>
+                </xacro:unless>
+                <xacro:if value="${is_light}">
+                    <parent link="link2_light"/>
+                </xacro:if>
+                <child link="camera_link"/>
+                <origin xyz="${l2/2} 0 ${h2-0.05}" rpy="${PI} 0 ${-PI/2}"/>
+            </joint>
+        </xacro:if>
         <!-- Joint 1 (Revolute) -->
         <joint name="joint1" type="revolute">

File: urdf/stereo_camera.sdf.xacro (robot description, xacro)
@@ -8,72 +8,81 @@
     <xacro:property name="hfov" value="${PI}/3" />
     <xacro:property name="name_prefix" value="/camera" />
-    <gazebo reference="camera_link">
-        <!-- left camera -->
-        <sensor name="left_camera_sensor" type="camera">
-            <always_on>1</always_on>
-            <update_rate>${fps}</update_rate>
-            <pose>0 0 0 0 0 0</pose>
-            <camera>
-                <horizontal_fov>${hfov}</horizontal_fov>
-                <image>
-                    <width>${width}</width>
-                    <height>${height}</height>
-                    <format>R8G8B8</format>
-                </image>
-                <clip>
-                    <near>0.1</near>
-                    <far>10.0</far>
-                </clip>
-            </camera>
-            <topic>${name_prefix}/left/image_raw</topic>
-        </sensor>
-        <!-- right camera -->
-        <sensor name="right_camera_sensor" type="camera">
-            <always_on>1</always_on>
-            <update_rate>${fps}</update_rate>
-            <pose>${baseline} 0 0 0 0 0</pose>
-            <camera>
-                <horizontal_fov>${hfov}</horizontal_fov>
-                <image>
-                    <width>${width}</width>
-                    <height>${height}</height>
-                    <format>R8G8B8</format>
-                </image>
-                <clip>
-                    <near>0.1</near>
-                    <far>10.0</far>
-                </clip>
-            </camera>
-            <topic>${name_prefix}/right/image_raw</topic>
-        </sensor>
-        <!-- depth -->
-        <sensor name="depth_sensor" type="depth">
-            <always_on>1</always_on>
-            <update_rate>${fps}</update_rate>
-            <pose>0 0 0 0 0 0</pose>
-            <camera>
-                <horizontal_fov>${hfov}</horizontal_fov>
-                <image>
-                    <width>${width}</width>
-                    <height>${height}</height>
-                    <format>R8G8B8</format>
-                </image>
-                <clip>
-                    <near>0.1</near>
-                    <far>10.0</far>
-                </clip>
-            </camera>
-            <topic>${name_prefix}/depth/image_raw</topic>
-        </sensor>
-        <!-- pointcloud -->
-        <sensor name="points_sensor" type="pointcloud">
-            <always_on>1</always_on>
-            <update_rate>${fps}</update_rate>
-            <pose>0 0 0 0 0 0</pose>
-            <pointcloud>
-                <render_mode>points</render_mode>
-            </pointcloud>
-            <topic>${name_prefix}/points</topic>
-        </sensor>
-    </gazebo>
+    <xacro:macro name="stereo_camera">
+        <link name="camera_sensor_link">
+            <!-- left camera -->
+            <sensor name="left_camera_sensor" type="camera">
+                <always_on>true</always_on>
+                <visualize>true</visualize>
+                <update_rate>${fps}</update_rate>
+                <pose>0 0 0 0 0 0</pose>
+                <camera>
+                    <horizontal_fov>${hfov}</horizontal_fov>
+                    <image>
+                        <width>${width}</width>
+                        <height>${height}</height>
+                        <format>R8G8B8</format>
+                    </image>
+                    <clip>
+                        <near>0.1</near>
+                        <far>10.0</far>
+                    </clip>
+                </camera>
+                <topic>${name_prefix}/left/image_raw</topic>
+            </sensor>
+            <!-- right camera -->
+            <sensor name="right_camera_sensor" type="camera">
+                <always_on>true</always_on>
+                <visualize>true</visualize>
+                <update_rate>${fps}</update_rate>
+                <pose>${baseline} 0 0 0 0 0</pose>
+                <camera>
+                    <horizontal_fov>${hfov}</horizontal_fov>
+                    <image>
+                        <width>${width}</width>
+                        <height>${height}</height>
+                        <format>R8G8B8</format>
+                    </image>
+                    <clip>
+                        <near>0.1</near>
+                        <far>10.0</far>
+                    </clip>
+                </camera>
+                <topic>${name_prefix}/right/image_raw</topic>
+            </sensor>
+            <!-- depth -->
+            <sensor name="depth_sensor" type="depth">
+                <always_on>true</always_on>
+                <visualize>true</visualize>
+                <update_rate>${fps}</update_rate>
+                <pose>0 0 0 0 0 0</pose>
+                <camera>
+                    <horizontal_fov>${hfov}</horizontal_fov>
+                    <image>
+                        <width>${width}</width>
+                        <height>${height}</height>
+                        <format>R8G8B8</format>
+                    </image>
+                    <clip>
+                        <near>0.1</near>
+                        <far>10.0</far>
+                    </clip>
+                </camera>
+                <topic>${name_prefix}/depth/image_raw</topic>
+            </sensor>
+            <!-- pointcloud -->
+            <!-- <sensor name="points_sensor" type="pointcloud">
+                <always_on>true</always_on>
+                <visualize>true</visualize>
+                <update_rate>${fps}</update_rate>
+                <pose>0 0 0 0 0 0</pose>
+                <pointcloud>
+                    <render_mode>points</render_mode>
+                </pointcloud>
+                <topic>${name_prefix}/points</topic>
+            </sensor> -->
+        </link>
+    </xacro:macro>
+    <model name="stereo_camera">
+        <xacro:stereo_camera/>
+    </model>
 </sdf>

File: urdf/weeder_robot.xacro (robot description, xacro)
@@ -4,6 +4,6 @@
     <!-- Parameters  -->
     <xacro:arg name= "is_light" default="true"/>
-    <xacro:arg name="use_camera" default="true"/>
     <xacro:arg name= "controller_yaml" default=""/>
+    <xacro:arg name= "use_camera" default="false"/>
     <xacro:macro name="weeder_robot" params="is_light use_camera controller_yaml">
         <!-- Including base and arm xacro files -->
@@ -13,5 +13,5 @@
         <xacro:bunker_fake/>
         <!-- Create robotic arm -->
-        <xacro:arm is_light="${is_light}"/>
+        <xacro:arm is_light="${is_light}" use_camera="${use_camera}"/>
         <!-- Create weeder robot by connecting base and arm -->
         <!-- Fixed joint connecting base_link and arm_base_link -->
@@ -47,10 +47,5 @@
             </sensor> -->
         </gazebo>
-        <!-- Add camera simulation -->
-        <xacro:if value="${use_camera}">
-            <xacro:include filename="$(find arm_mazzolini)/urdf/stereo_camera.sdf.xacro"/>
-            <xacro:stereo_camera/>
-        </xacro:if>
     </xacro:macro>
-    <xacro:weeder_robot is_light="$(arg is_light)" controller_yaml="$(arg controller_yaml)"/>
+    <xacro:weeder_robot is_light="$(arg is_light)" use_camera="$(arg use_camera)" controller_yaml="$(arg controller_yaml)"/>
 </robot>

Commit message: added dalyed spawner for controllers

File: urdf/arm.xacro (robot description, xacro)
@@ -1,5 +1,5 @@
 <?xml version="1.0"?>
 <robot name="weeder_robot" xmlns:xacro="http://www.ros.org/wiki/xacro">
-    <!-- Parameters -->
+    <!-- Arm Parameters -->
     <xacro:property name="PI" value="3.141592" />
     <xacro:property name="base_mesh" value="file://$(find arm_mazzolini)/meshes/stl/Arm_base.stl"/>
@@ -15,5 +15,5 @@
     <xacro:property name="l2" value="0.250"/>
     <xacro:property name="scale" value="1e-3 1e-3 1e-3"/>
-    <xacro:macro name="arm" params= "is_light use_camera">
+    <xacro:macro name="arm" params= "is_light">
         <!-- Base Link of robotic arm-->
         <link name="arm_base_link">
@@ -113,30 +113,6 @@
                                                                     izz="0.012756684"
                     />
-                    </inertial>
+                </inertial>
             </link>
-        </xacro:if>
-        <xacro:if value="${use_camera}">
-            <link name="camera_link">
-                <visual>
-                    <geometry>
-                        <mesh filename="${camera_mesh}" scale="${scale}*1000"/>
-                    </geometry>
-                </visual>
-                <collision>
-                    <geometry>
-                        <mesh filename="${camera_mesh}" scale="${scale}*1000"/>
-                    </geometry>
-                </collision>
-            </link>
-            <joint name="camera_joint" type="fixed">
-                <xacro:unless value="${is_light}">
-                    <parent link="link2_heavy"/>
-                </xacro:unless>
-                <xacro:if value="${is_light}">
-                    <parent link="link2_light"/>
-                </xacro:if>
-                <child link="camera_link"/>
-                <origin xyz="${l2/2} 0 ${h2-0.05}" rpy="${PI} 0 ${-PI/2}"/>
-            </joint>
         </xacro:if>
         <!-- Joint 1 (Revolute) -->
@@ -163,4 +139,5 @@
         </joint>
     </xacro:macro>
+    <!-- Do not add plugins here -->
     <xacro:macro name="joint_control" params="name">
         <joint name="${name}">

File: urdf/bunker_fake.xacro (robot description, xacro)
@@ -124,4 +124,5 @@
         <xacro:bunker_wheel name="rear_right_wheel" pos_x="-${wheel_pos_x}" pos_y="-${wheel_pos_y}"/>
     </xacro:macro>
+    <!-- Do not add plugins here -->
     <xacro:macro name="wheel_control" params="name">
         <joint name="${name}_joint">

File: urdf/stereo_camera.sdf.xacro (robot description, xacro)
@@ -6,7 +6,8 @@
     <xacro:property name="height" value="720" />
     <xacro:property name="fps" value="30" />
-    <xacro:property name="hfov" value="${PI}/3" />
+    <xacro:property name="hfov" value="${PI/3}" />
     <xacro:property name="name_prefix" value="/camera" />
     <xacro:macro name="stereo_camera">
+        <static>true</static>
         <link name="camera_sensor_link">
             <!-- left camera -->

File: urdf/weeder_robot.xacro (robot description, xacro)
@@ -6,12 +6,14 @@
     <xacro:arg name= "controller_yaml" default=""/>
     <xacro:arg name= "use_camera" default="false"/>
-    <xacro:macro name="weeder_robot" params="is_light use_camera controller_yaml">
+    <xacro:arg name= "use_sim_time" default="true"/>
+    <xacro:macro name="weeder_robot" params="is_light use_camera controller_yaml use_sim_time">
         <!-- Including base and arm xacro files -->
         <xacro:include filename="$(find arm_mazzolini)/urdf/bunker_fake.xacro"/>
         <xacro:include filename="$(find arm_mazzolini)/urdf/arm.xacro"/>
+        <xacro:include filename="$(find arm_mazzolini)/urdf/camera.xacro"/>
         <!-- Create base -->
         <xacro:bunker_fake/>
         <!-- Create robotic arm -->
-        <xacro:arm is_light="${is_light}" use_camera="${use_camera}"/>
+        <xacro:arm is_light="${is_light}"/>
         <!-- Create weeder robot by connecting base and arm -->
         <!-- Fixed joint connecting base_link and arm_base_link -->
@@ -21,4 +23,8 @@
             <origin xyz="0 -0.3 0.28" rpy="0 0 -${PI/2}"/>
         </joint>
+        <!-- Include depth camera if requested -->
+        <xacro:if value="${use_camera}">
+            <xacro:depth_camera is_light="${is_light}" use_sim_time="${use_sim_time}"/>
+        </xacro:if>
         <!-- Ros2 Control -->
         <ros2_control name="weeder_controller" type="system">
@@ -34,4 +40,5 @@
         </ros2_control>
         <!-- Gazebo Plugins -->
+        <!-- TODO: Change plugins if changing Gazebo version -->
         <gazebo>
             <plugin filename="gz_ros2_control-system" name="gz_ros2_control::GazeboSimROS2ControlPlugin">
@@ -48,4 +55,4 @@
         </gazebo>
     </xacro:macro>
-    <xacro:weeder_robot is_light="$(arg is_light)" use_camera="$(arg use_camera)" controller_yaml="$(arg controller_yaml)"/>
+    <xacro:weeder_robot is_light="$(arg is_light)" use_camera="$(arg use_camera)" controller_yaml="$(arg controller_yaml)" use_sim_time="$(arg use_sim_time)"/>
 </robot>

Commit message: added ExG and ExGR for image analysis

File: urdf/arm.xacro (robot description, xacro)
@@ -116,4 +116,32 @@
             </link>
         </xacro:if>
+        <!-- Laser -->
+        <link name="laser">
+            <visual>
+                <geometry>
+                    <cylinder radius="0.005" length="1.0"/>
+                </geometry>
+                <material name="grey">
+                    <color rgba="0.6 0.6 0.6 1"/>
+                </material>
+            </visual>
+        </link>
+        <joint name="laser_joint" type="fixed">
+            <xacro:if value="${is_light}">
+                <parent link="link2_light"/>
+            </xacro:if>
+            <xacro:unless value="${is_light}">
+                <parent link="link2_heavy"/>
+            </xacro:unless>
+            <child link="laser"/>
+            <origin xyz="${l2} 0 ${-h2-0.5}" rpy="0 0 0"/>
+        </joint>
+        <link name="kinematic_link">
+        </link>
+        <joint name="fixed_for_kinematic" type="fixed">
+            <parent link="arm_base_link"/>
+            <child link="kinematic_link"/>
+            <origin xyz="${l0} 0 ${h0}" rpy="0 0 0"/>
+        </joint>
         <!-- Joint 1 (Revolute) -->
         <joint name="joint1" type="revolute">

File: urdf/camera.xacro (robot description, xacro)
@@ -25,5 +25,5 @@
                     <mesh filename="${camera_mesh}" scale="${scale}"/>
                 </geometry>
-                <origin xyz="0 0 -0.07" rpy="0 0 0"/>
+                <origin xyz="0 0 0" rpy="0 0 0"/>
             </collision>
             <inertial>
@@ -44,5 +44,11 @@
             </xacro:if>
             <child link="camera_link"/>
-            <origin xyz="${l2/2} 0 ${-h2-0.03}" rpy="${PI+PI/9} 0 ${-PI/2}"/>
+            <origin xyz="${l2/3} 0 ${-h2-0.03}" rpy="${PI+PI/9} 0 ${-PI/2}"/>
+        </joint>
+        <link name="camera_kinematic"/>
+        <joint name="camera_kinematic_joint" type="fixed">
+            <parent link="camera_link"/>
+            <child link="camera_kinematic"/>
+            <origin xyz="0 0 0.03" rpy="0 0 0"/>
         </joint>
         <link name="camera_optical_frame"/>
@@ -52,5 +58,5 @@
                 <parent link="camera_link"/>
                 <child link="camera_optical_frame"/>
-                <origin xyz="0 0 0.07" rpy="${PI/2} ${-PI/2} 0"/>
+                <origin xyz="0 0 0.03" rpy="${PI/2} ${-PI/2} 0"/>
             </joint>
         </xacro:if>

File: urdf/weeder_robot.xacro (robot description, xacro)
@@ -53,4 +53,11 @@
                 <topic>force_torque_sensor</topic>
             </sensor> -->
+            <plugin
+                filename="libignition-gazebo-pose-publisher-system.so"
+                name="ignition::gazebo::systems::PosePublisher">
+                <publish_model_pose>true</publish_model_pose>
+                <publish_link_pose>false</publish_link_pose>
+                <update_frequency>50</update_frequency>
+            </plugin>
         </gazebo>
     </xacro:macro>
