Commit message: Changed textures to match real robot

File: urdf/arm.xacro (robot description, xacro)
@@ -5,14 +5,17 @@
     <xacro:property name="base_mesh" value="file://$(find arm_mazzolini)/meshes/stl/Arm_base.stl"/>
     <xacro:property name="link1_mesh" value="file://$(find arm_mazzolini)/meshes/stl/Braccio_intermedio.stl"/>
-    <xacro:property name="link2_heavy_mesh" value="file://$(find arm_mazzolini)/meshes/stl/Braccio2.stl"/>
-    <xacro:property name="link2_light_mesh" value="file://$(find arm_mazzolini)/meshes/stl/Braccio3.stl"/>
-    <xacro:property name="camera_mesh" value="file://$(find arm_mazzolini)/meshes/stl/D435.stl"/>
-    <xacro:property name="h0" value="0.07"/>
+    <xacro:property name="link2_heavy_mesh" value="file://$(find arm_mazzolini)/meshes/stl/Assieme_ee_heavy_partial.stl"/>
+    <xacro:property name="link2_light_mesh" value="file://$(find arm_mazzolini)/meshes/stl/Assieme_ee_light_partial.stl"/>
+    <xacro:property name="ee_light_mesh" value="file://$(find arm_mazzolini)/meshes/stl/ee_laser_light.stl"/>
+    <xacro:property name="ee_heavy_mesh" value="file://$(find arm_mazzolini)/meshes/stl/ee_laser_heavy.stl"/>
+    <!-- <xacro:property name="camera_mesh" value="file://$(find arm_mazzolini)/meshes/stl/D435.stl"/> -->
+    <xacro:property name="h0" value="0.065"/>
     <xacro:property name="l0" value="0.190"/>
     <xacro:property name="h1" value="0.0"/>
     <xacro:property name="l1" value="0.190"/>
-    <xacro:property name="h2" value="-0.037"/>
+    <xacro:property name="h2" value="0.03"/>
     <xacro:property name="l2" value="0.250"/>
     <xacro:property name="scale" value="1e-3 1e-3 1e-3"/>
+    <xacro:property name="no_scale" value="1.0 1.0 1.0"/>
     <xacro:macro name="arm" params= "is_light">
         <!-- Base Link of robotic arm-->
@@ -46,6 +49,6 @@
                     <mesh filename="${link1_mesh}" scale="${scale}"/>
                 </geometry>
-                <material name="blue">
-                    <color rgba="0.2 0.2 0.8 1"/>
+                <material name="grey">
+                    <color rgba="0.6 0.6 0.6 1"/>
                 </material>
             </visual>
@@ -58,7 +61,7 @@
                 <origin xyz="${l1/2} 0 ${h1/2}" rpy="0 0 0"/>
                 <mass value="0.220"/>
-            <inertia ixx="0.000162936"    ixy="-0.000002254"   ixz="0.000291499"
-                                            iyy="0.002971043"    iyz="0.0"
-                                                                izz="0.002927669"
+            <inertia ixx="0.000162936"  ixy="-0.000002254"  ixz="0.000291499"
+                                        iyy="0.002971043"   iyz="0.0"
+                                                            izz="0.002927669"
                 />
             </inertial>
@@ -69,24 +72,52 @@
                 <visual>
                     <geometry>
-                        <mesh filename="${link2_heavy_mesh}" scale="${scale}"/>
-                    </geometry>
-                    <material name="green">
-                        <color rgba="0.2 0.8 0.2 1"/>
-                    </material>
-                </visual>
-                <collision>
-                    <geometry>
-                        <mesh filename="${link2_heavy_mesh}" scale="${scale}"/>
-                    </geometry>
-                </collision>
-                <inertial>
-                    <origin xyz="${l2/2} 0 ${h2/2}"  rpy="0 0 0"/>
-                    <mass value="1.701"/>
-                    <inertia ixx="0.011472444"   ixy="0.0"           ixz="-0.024108120"
-                                                iyy="0.104552446"   iyz="0.0"
-                                                                    izz="0.094998962"
-                    />
-                </inertial>
-            </link>
+                        <mesh filename="${link2_heavy_mesh}" scale="${no_scale}"/>
+                    </geometry>
+                    <material name="grey">
+                        <color rgba="0.6 0.6 0.6 1"/>
+                    </material>
+                </visual>
+                <collision>
+                    <geometry>
+                        <mesh filename="${link2_heavy_mesh}" scale="${no_scale}"/>
+                    </geometry>
+                </collision>
+                <inertial>
+                    <origin xyz="0.1153 0 0.0235"  rpy="0 0 0"/>
+                    <mass value="0.845"/>
+                    <inertia ixx="0.000709911"  ixy="0.0"           ixz="0.00002662"
+                                                iyy="0.006001619"   iyz="0.0"
+                                                                    izz="0.006511388"
+                    />
+                </inertial>
+            </link>
+            <link name="end_effector">
+                <visual>
+                    <geometry>
+                        <mesh filename="${ee_heavy_mesh}" scale="${no_scale}"/>
+                    </geometry>
+                    <material name="black">
+                        <color rgba="0.1 0.1 0.1 1"/>
+                    </material>
+                </visual>
+                <collision>
+                    <geometry>
+                        <mesh filename="${ee_heavy_mesh}" scale="${no_scale}"/>
+                    </geometry>
+                </collision>
+                <inertial>
+                    <origin xyz="0 0 0.108" rpy="0 0 0"/>
+                    <mass value="1.549"/>
+                    <inertia ixx="0.005320713"  ixy="0.0"           ixz="0.0"
+                                                iyy="0.005320713"   iyz="0.0"
+                                                                    izz="0.001627615"
+                    />
+                </inertial>
+            </link>
+            <joint name="end_effector_joint" type="fixed">
+                <parent link="link2_heavy"/>
+                <child link="end_effector"/>
+                <origin xyz="${l2} 0 -${h2}" rpy="0 0 0"/>
+            </joint>
         </xacro:unless>
         <!-- Link 2 with IPG head -->
@@ -95,24 +126,52 @@
                 <visual>
                     <geometry>
-                        <mesh filename="${link2_light_mesh}" scale="${scale}"/>
-                    </geometry>
-                    <material name="green">
-                        <color rgba="0.2 0.8 0.2 1"/>
-                    </material>
-                </visual>
-                <collision>
-                    <geometry>
-                        <mesh filename="${link2_light_mesh}" scale="${scale}"/>
-                    </geometry>
-                </collision>
-                <inertial>
-                    <origin xyz="${l2/2} 0 ${h2/2}" rpy="0 0 0"/>
-                    <mass value="1.701"/>
-                    <inertia ixx="0.00490436"   ixy="0.0"           ixz="-0.001747695"
-                                                iyy="0.013178423"    iyz="0.0"
-                                                                    izz="0.012756684"
-                    />
-                </inertial>
-            </link>
+                        <mesh filename="${link2_light_mesh}" scale="${no_scale}"/>
+                    </geometry>
+                    <material name="grey">
+                        <color rgba="0.6 0.6 0.6 1"/>
+                    </material>
+                </visual>
+                <collision>
+                    <geometry>
+                        <mesh filename="${link2_light_mesh}" scale="${no_scale}"/>
+                    </geometry>
+                </collision>
+                <inertial>
+                    <origin xyz="0.0888 0 0.0243" rpy="0 0 0"/>
+                    <mass value="0.704"/>
+                    <inertia ixx="0.000401870"  ixy="0.0"           ixz="-0.000064005"
+                                                iyy="0.002700823"   iyz="0.0"
+                                                                    izz="0.002965740"
+                    />
+                </inertial>
+            </link>
+            <link name="end_effector">
+                <visual>
+                    <geometry>
+                        <mesh filename="${ee_light_mesh}" scale="${no_scale}"/>
+                    </geometry>
+                    <material name="black">
+                        <color rgba="0.1 0.1 0.1 1"/>
+                    </material>
+                </visual>
+                <collision>
+                    <geometry>
+                        <mesh filename="${ee_light_mesh}" scale="${no_scale}"/>
+                    </geometry>
+                </collision>
+                <inertial>
+                    <origin xyz="0 0 0.0686" rpy="0 0 0"/>
+                    <mass value="0.096"/>
+                    <inertia ixx="0.0001466"    ixy="0.0"       ixz="0.0"
+                                                iyy="0.0001466" iyz="0.0"
+                                                                izz="0.0000102"
+                    />
+                </inertial>
+            </link>
+            <joint name="end_effector_joint" type="fixed">
+                <parent link="link2_light"/>
+                <child link="end_effector"/>
+                <origin xyz="${l2} 0 -0.037" rpy="0 0 0"/>
+            </joint>
         </xacro:if>
         <!-- Laser -->
@@ -123,7 +182,9 @@
                 </geometry>
                 <material name="grey">
-                    <color rgba="0.6 0.6 0.6 1"/>
+                    <color rgba="0.6 0.6 0.6 0.9"/>
                 </material>
             </visual>
+        </link>
+        <link name="kinematic_link">
         </link>
         <joint name="laser_joint" type="fixed">
@@ -135,8 +196,6 @@
             </xacro:unless>
             <child link="laser"/>
-            <origin xyz="${l2} 0 ${-h2-0.5}" rpy="0 0 0"/>
-        </joint>
-        <link name="kinematic_link">
-        </link>
+            <origin xyz="${l2} 0 ${h2-0.5}" rpy="0 0 0"/>
+        </joint>
         <joint name="fixed_for_kinematic" type="fixed">
             <parent link="arm_base_link"/>

File: urdf/bunker_fake.xacro (robot description, xacro)
@@ -3,49 +3,53 @@
     <xacro:macro name="bunker_fake">
         <xacro:property name="PI" value="3.141592" />
-        <!-- <xacro:property name="mesh_path" value="file://$(find arm_mazzolini)/meshes/bunker"/> -->
-        <xacro:property name="base_mass" value="180"/>
+        <xacro:property name="bunker_fake_mesh" value="file://$(find arm_mazzolini)/meshes/stl/Bunker_fake_v2.stl"/>
+        <xacro:property name="base_mass" value="130"/>
+        <xacro:property name="box_size_x" value="0.852"/>
+        <xacro:property name="box_size_y" value="0.545"/>
+        <xacro:property name="box_size_z" value="0.400"/>
         <xacro:property name="wheel_mass" value="5"/>
-        <xacro:property name="wheel_radius" value="0.2"/>
+        <xacro:property name="wheel_radius" value="0.18"/>
         <xacro:property name="wheel_length" value="0.15"/>
-        <xacro:property name="wheel_pos_x" value="0.45"/>
-        <xacro:property name="wheel_pos_y" value="0.5"/>
+        <xacro:property name="wheel_pos_x" value="${(box_size_x - 2*wheel_radius)/2+0.2}"/>
+        <xacro:property name="wheel_pos_y" value="${(box_size_y + wheel_length)/2}"/>
+        <xacro:property name="wheel_pos_z" value="${0.465 - box_size_z - wheel_radius}"/>
+        <link name="base_link"/>
         <link
             name="inertial">
             <inertial>
             <origin
-                xyz="0.0 0.0 0.0"
-                rpy="0 0 0" />
-            <mass
-                value="${base_mass}" />
-            <inertia
-                ixx="15.7"
-                ixy="0.0"
-                ixz="0.0"
-                iyy="26.0"
-                iyz="0.0"
-                izz="33.42" />
+                    xyz="0.0 0.0 0.0"
+                    rpy="0 0 0" />
+                <mass
+                    value="${base_mass}" />
+                <inertia
+                    ixx="15.7"
+                    ixy="0.0"
+                    ixz="0.0"
+                    iyy="26.0"
+                    iyz="0.0"
+                    izz="33.42" />
             </inertial>
             <visual>
-            <origin
-                xyz="0.0 0.0 0.0"
-                rpy="0 0 0" />
-            <geometry>
-                <box size="1.08 0.785 0.47" />
-            </geometry>
-            <material
-                name="">
-                <color
-                rgba="0.5 0.5 0.5 1" />
-            </material>
+                <origin
+                    xyz="0.0 0.0 ${-box_size_z/2-0.065}"
+                    rpy="0 0 0" />
+                <geometry>
+                    <mesh filename="${bunker_fake_mesh}" />
+                    <!-- <box size="${box_size_x} ${box_size_y} ${box_size_z}" /> -->
+                </geometry>
+                <material
+                    name="">
+                    <color
+                    rgba="0.5 0.5 0.5 1" />
+                </material>
             </visual>
             <collision>
-            <origin
-                xyz="0.0 0.0 0.0" rpy="0.0 0.0 0.0" />
-            <geometry>
-                <box size="1.08 0.785 0.47" />
-            </geometry>
+                <origin
+                    xyz="0.0 0.0 0.0" rpy="0.0 0.0 0.0" />
+                <geometry>
+                    <box size="${box_size_x} ${box_size_y} ${box_size_z}" />
+                </geometry>
             </collision>
-        </link>
-        <link name="base_link">
         </link>
         <joint
@@ -70,35 +74,35 @@
                     value="${wheel_mass}" />
                 <inertia
-                    ixx="${wheel_mass*(wheel_radius*wheel_radius/4 + wheel_length*wheel_length/12)}"
+                    ixx="${wheel_mass*wheel_radius*wheel_radius/2}"
                     ixy="0.0"
                     ixz="0.0"
                     iyy="${wheel_mass*(wheel_radius*wheel_radius/4 + wheel_length*wheel_length/12)}"
                     iyz="0.0"
-                    izz="${wheel_mass*wheel_radius*wheel_radius/2}" />
+                    izz="${wheel_mass*(wheel_radius*wheel_radius/4 + wheel_length*wheel_length/12)}" />
                 </inertial>
-                <visual>
-                <origin
-                    xyz="0.0 0.0 0.0"
-                    rpy="${PI/2} 0 0" />
-                <geometry>
-                    <cylinder
-                    radius="${wheel_radius}"
-                    length="${wheel_length}" />
-                </geometry>
-                <material
-                    name="">
-                    <color
-                    rgba="0.5 0.5 0.5 1" />
-                </material>
-                </visual>
+                <!-- <visual>
+                    <origin
+                        xyz="0.0 0.0 0.0"
+                        rpy="${PI/2} 0 0" />
+                    <geometry>
+                        <cylinder
+                        radius="${wheel_radius}"
+                        length="${wheel_length}" />
+                    </geometry>
+                    <material
+                        name="">
+                        <color
+                        rgba="0.5 0.5 0.5 1" />
+                    </material>
+                </visual> -->
                 <collision>
-                <origin
-                    xyz="0.0 0.0 0.0"
-                    rpy="${PI/2} 0 0" />
-                <geometry>
-                    <cylinder
-                    radius="${wheel_radius}"
-                    length="${wheel_length}" />
-                </geometry>
+                    <origin
+                        xyz="0.0 0.0 0.0"
+                        rpy="${PI/2} 0 0" />
+                    <geometry>
+                        <cylinder
+                        radius="${wheel_radius}"
+                        length="${wheel_length}" />
+                    </geometry>
                 </collision>
             </link>
@@ -109,13 +113,9 @@
                     link="${name}" />
                 <origin
-                    xyz="${pos_x} ${pos_y} -0.12"
+                    xyz="${pos_x} ${pos_y} ${wheel_pos_z}"
                     rpy="0 0 0" />
                 <axis
                     xyz="0 1 0" />
             </joint>
-            <!-- <gazebo reference="${name}">
-                <mu1>1.0</mu1>
-                <mu2>1.0</mu2>
-            </gazebo> -->
         </xacro:macro>
         <xacro:bunker_wheel name="front_left_wheel" pos_x="${wheel_pos_x}" pos_y="${wheel_pos_y}"/>

File: urdf/camera.xacro (robot description, xacro)
@@ -9,31 +9,9 @@
     <xacro:property name="hfov" value="${PI/3}" />
     <xacro:property name="name_prefix" value="/simulated_D435" />
+    <xacro:property name="l_camera" value="0.06185"/>
+    <xacro:property name="h_camera" value="0.0083"/>
     <!-- TODO: This file is valid only in simulation, change use_sim_time if condition -->
     <xacro:macro name="depth_camera" params= "is_light use_sim_time">
-        <link name="camera_link">
-            <visual>
-                <geometry>
-                    <mesh filename="${camera_mesh}" scale="${scale}"/>
-                </geometry>
-                <material name="grey">
-                    <color rgba="0.6 0.6 0.6 1"/>
-                </material>
-                <origin xyz="0 0 0" rpy="0 0 0"/>
-            </visual>
-            <collision>
-                <geometry>
-                    <mesh filename="${camera_mesh}" scale="${scale}"/>
-                </geometry>
-                <origin xyz="0 0 0" rpy="0 0 0"/>
-            </collision>
-            <inertial>
-                <origin xyz="0 0 0" rpy="0 0 0"/>
-                <mass value="0.072"/>
-                <inertia ixx="0.000005"   ixy="0.0"           ixz="0.00000"
-                                            iyy="0.000005"    iyz="0.0"
-                                                                izz="0.000005"
-                />
-            </inertial>
-        </link>
+        <link name="camera_link"/>
         <joint name="camera_joint" type="fixed">
             <xacro:unless value="${is_light}">
@@ -44,5 +22,5 @@
             </xacro:if>
             <child link="camera_link"/>
-            <origin xyz="${l2/3} 0 ${-h2-0.03}" rpy="${PI+PI/18} 0 ${-PI/2}"/>
+            <origin xyz="${l_camera} 0 ${h_camera}" rpy="${PI+PI/10} 0 ${-PI/2}"/>
         </joint>
         <link name="camera_kinematic"/>
@@ -50,5 +28,5 @@
             <parent link="camera_link"/>
             <child link="camera_kinematic"/>
-            <origin xyz="0 0 0.03" rpy="0 0 0"/>
+            <origin xyz="0 0 0.0" rpy="0 0 0"/>
         </joint>
         <link name="camera_optical_frame"/>
@@ -58,5 +36,5 @@
                 <parent link="camera_link"/>
                 <child link="camera_optical_frame"/>
-                <origin xyz="0 0 0.03" rpy="${PI/2} ${-PI/2} 0"/>
+                <origin xyz="0 0 0.003" rpy="${PI/2} ${-PI/2} 0"/>
             </joint>
         </xacro:if>

File: urdf/weeder_robot.xacro (robot description, xacro)
@@ -21,5 +21,5 @@
             <parent link="base_link"/>
             <child link="arm_base_link"/>
-            <origin xyz="0 -0.3 0.28" rpy="0 0 -${PI/2}"/>
+            <origin xyz="0 -0.3 0.23" rpy="0 0 -${PI/2}"/>
         </joint>
         <!-- Include depth camera if requested -->
