Commit message: Tuned gains

File: urdf/arm.xacro (robot description, xacro)
@@ -10,5 +10,5 @@
     <xacro:property name="ee_heavy_mesh" value="file://$(find arm_mazzolini)/meshes/stl/ee_laser_heavy.stl"/>
     <!-- <xacro:property name="camera_mesh" value="file://$(find arm_mazzolini)/meshes/stl/D435.stl"/> -->
-    <xacro:property name="h0" value="0.065"/>
+    <xacro:property name="h0" value="0.07"/>
     <xacro:property name="l0" value="0.190"/>
     <xacro:property name="h1" value="0.0"/>
@@ -37,7 +37,7 @@
                 <origin xyz="0 0 0" rpy="0 0 0"/>
                 <mass value="2.074"/>
-            <inertia ixx="0.006004333"  ixy="0.000070425"   ixz="0.001686871"
-                                        iyy="0.010804985"   iyz="-0.000043204"
-                                                            izz="0.013471098"
+            <inertia ixx="0.006004333"  ixy="0.0"           ixz="-0.000283467"
+                                        iyy="0.0.0628431"   iyz="0.0"
+                                                            izz="0.010101581"
                 />
             </inertial>
@@ -61,7 +61,7 @@
                 <origin xyz="${l1/2} 0 ${h1/2}" rpy="0 0 0"/>
                 <mass value="0.220"/>
-            <inertia ixx="0.000162936"  ixy="-0.000002254"  ixz="0.000291499"
-                                        iyy="0.002971043"   iyz="0.0"
-                                                            izz="0.002927669"
+            <inertia ixx="0.000143696"  ixy="0.0"           ixz="0.000134444"
+                                        iyy="0.001669532"   iyz="0.0"
+                                                            izz="0.001645390"
                 />
             </inertial>
@@ -210,5 +210,5 @@
             <!-- <origin xyz="0 0 ${h0}" rpy="0 0 0"/> -->
             <axis xyz="0 0 1"/>
-            <limit effort="100" lower="-${PI}" upper="${PI}" velocity="1000"/>
+            <limit effort="1000" lower="-${PI}" upper="${PI}" velocity="100"/>
         </joint>
         <!-- Joint 2 (Revolute) -->
@@ -223,5 +223,5 @@
             <origin xyz="${l1} 0 ${h1}" rpy="0 0 0"/>
             <axis xyz="0 0 1"/>
-            <limit effort="100" lower="-${PI}" upper="${PI}" velocity="1000"/>
+            <limit effort="1000" lower="-${PI}" upper="${PI}" velocity="100"/>
         </joint>
     </xacro:macro>

File: urdf/bunker_fake.xacro (robot description, xacro)
@@ -11,5 +11,5 @@
         <xacro:property name="wheel_radius" value="0.18"/>
         <xacro:property name="wheel_length" value="0.15"/>
-        <xacro:property name="wheel_pos_x" value="${(box_size_x - 2*wheel_radius)/2+0.2}"/>
+        <xacro:property name="wheel_pos_x" value="${box_size_x/2}"/>
         <xacro:property name="wheel_pos_y" value="${(box_size_y + wheel_length)/2}"/>
         <xacro:property name="wheel_pos_z" value="${0.465 - box_size_z - wheel_radius}"/>
@@ -74,8 +74,8 @@
                     value="${wheel_mass}" />
                 <inertia
-                    ixx="${wheel_mass*wheel_radius*wheel_radius/2}"
+                    ixx="${wheel_mass*(wheel_radius*wheel_radius/4 + wheel_length*wheel_length/12)}"
                     ixy="0.0"
                     ixz="0.0"
-                    iyy="${wheel_mass*(wheel_radius*wheel_radius/4 + wheel_length*wheel_length/12)}"
+                    iyy="${wheel_mass*wheel_radius*wheel_radius/2}"
                     iyz="0.0"
                     izz="${wheel_mass*(wheel_radius*wheel_radius/4 + wheel_length*wheel_length/12)}" />
@@ -117,5 +117,14 @@
                 <axis
                     xyz="0 1 0" />
+                <limit effort="10000" velocity="100"/>
+                <dynamics damping="0.1" friction="0.0"/>
             </joint>
+            <gazebo reference="${name}">
+                <mu1>3.0</mu1>
+                <mu2>1.0</mu2>
+                <kp>10000.0</kp>
+                <kd>10.0</kd>
+                <minDepth>0.001</minDepth>
+            </gazebo>
         </xacro:macro>
         <xacro:bunker_wheel name="front_left_wheel" pos_x="${wheel_pos_x}" pos_y="${wheel_pos_y}"/>

File: urdf/weeder_robot.xacro (robot description, xacro)
@@ -21,5 +21,5 @@
             <parent link="base_link"/>
             <child link="arm_base_link"/>
-            <origin xyz="0 -0.3 0.23" rpy="0 0 -${PI/2}"/>
+            <origin xyz="0 -0.3 0.235" rpy="0 0 -${PI/2}"/>
         </joint>
         <!-- Include depth camera if requested -->

Commit message: added custom Gazebo launch file (silent)

File: urdf/arm.xacro (robot description, xacro)
@@ -38,5 +38,5 @@
                 <mass value="2.074"/>
             <inertia ixx="0.006004333"  ixy="0.0"           ixz="-0.000283467"
-                                        iyy="0.0.0628431"   iyz="0.0"
+                                        iyy="0.00628431"    iyz="0.0"
                                                             izz="0.010101581"
                 />
@@ -179,8 +179,8 @@
             <visual>
                 <geometry>
-                    <cylinder radius="0.005" length="1.0"/>
-                </geometry>
-                <material name="grey">
-                    <color rgba="0.6 0.6 0.6 0.9"/>
+                    <cylinder radius="0.002" length="1.0"/>
+                </geometry>
+                <material name="red">
+                    <color rgba="0.9 0 0 1"/>
                 </material>
             </visual>

File: urdf/camera.xacro (robot description, xacro)
@@ -28,5 +28,5 @@
             <parent link="camera_link"/>
             <child link="camera_kinematic"/>
-            <origin xyz="0 0 0.0" rpy="0 0 0"/>
+            <origin xyz="0 0 0" rpy="0 0 0"/>
         </joint>
         <link name="camera_optical_frame"/>
@@ -36,5 +36,5 @@
                 <parent link="camera_link"/>
                 <child link="camera_optical_frame"/>
-                <origin xyz="0 0 0.003" rpy="${PI/2} ${-PI/2} 0"/>
+                <origin xyz="0 0 0" rpy="${PI/2} ${-PI/2} 0"/>
             </joint>
         </xacro:if>
@@ -71,5 +71,6 @@
                     <width>${width}</width>
                     <height>${height}</height>
-                    <format>L8</format>
+                    <!-- <format>L8</format> -->
+                    <format>RGB_INT8</format>
                 </image>
                 <clip>

File: urdf/weeder_robot.xacro (robot description, xacro)
@@ -57,5 +57,5 @@
                 name="ignition::gazebo::systems::PosePublisher">
                 <publish_model_pose>true</publish_model_pose>
-                <publish_link_pose>false</publish_link_pose>
+                <publish_link_pose>true</publish_link_pose>
                 <update_frequency>20</update_frequency>
             </plugin>

Commit message: Added new world

File: urdf/arm.xacro (robot description, xacro)
@@ -176,5 +176,5 @@
         </xacro:if>
         <!-- Laser -->
-        <link name="laser">
+        <!-- <link name="laser">
             <visual>
                 <geometry>
@@ -185,6 +185,4 @@
                 </material>
             </visual>
-        </link>
-        <link name="kinematic_link">
         </link>
         <joint name="laser_joint" type="fixed">
@@ -197,5 +195,7 @@
             <child link="laser"/>
             <origin xyz="${l2} 0 ${h2-0.5}" rpy="0 0 0"/>
-        </joint>
+        </joint> -->
+        <link name="kinematic_link">
+        </link>
         <joint name="fixed_for_kinematic" type="fixed">
             <parent link="arm_base_link"/>

File: urdf/camera.xacro (robot description, xacro)
@@ -76,10 +76,12 @@
                 <clip>
                     <near>0.01</near>
-                    <far>30.0</far>
+                    <!-- <far>30.0</far> -->
+                     <far>5.0</far>
                 </clip>
                 <depth_camera>
                     <clip>
                     <near>0.1</near>
-                    <far>10.0</far>
+                    <!-- <far>10.0</far> -->
+                     <far>2.0</far>
                     </clip>
                 </depth_camera>

Commit message: Added YOLO network for plant recognition

File: urdf/arm.xacro (robot description, xacro)
@@ -176,6 +176,8 @@
         </xacro:if>
         <!-- Laser -->
-        <!-- <link name="laser">
+         <!-- Do not remove laser link, remove visual if needed -->
+        <link name="laser">
             <visual>
+                <origin xyz="0 0 -0.5" rpy="0 0 0"/>
                 <geometry>
                     <cylinder radius="0.002" length="1.0"/>
@@ -194,6 +196,6 @@
             </xacro:unless>
             <child link="laser"/>
-            <origin xyz="${l2} 0 ${h2-0.5}" rpy="0 0 0"/>
-        </joint> -->
+            <origin xyz="${l2} 0 ${h2}" rpy="0 0 0"/>
+        </joint>
         <link name="kinematic_link">
         </link>

File: urdf/camera.xacro (robot description, xacro)
@@ -11,7 +11,6 @@
     <xacro:property name="l_camera" value="0.06185"/>
     <xacro:property name="h_camera" value="0.0083"/>
-    <!-- TODO: This file is valid only in simulation, change use_sim_time if condition -->
-    <xacro:macro name="depth_camera" params= "is_light use_sim_time">
-        <link name="camera_link"/>
+    <xacro:macro name="depth_camera" params= "is_light">
+        <link name="camera_kinematic"/>
         <joint name="camera_joint" type="fixed">
             <xacro:unless value="${is_light}">
@@ -21,29 +20,14 @@
                 <parent link="link2_light"/>
             </xacro:if>
-            <child link="camera_link"/>
+            <child link="camera_kinematic"/>
             <origin xyz="${l_camera} 0 ${h_camera}" rpy="${PI+PI/10} 0 ${-PI/2}"/>
         </joint>
-        <link name="camera_kinematic"/>
-        <joint name="camera_kinematic_joint" type="fixed">
-            <parent link="camera_link"/>
-            <child link="camera_kinematic"/>
-            <origin xyz="0 0 0" rpy="0 0 0"/>
+        <link name="camera_optical_frame"/>
+        <!-- this joint rotates camera because Gazebo uses YZ plane instead of XY -->
+        <joint name="camera_optical_joint" type="fixed">
+            <parent link="camera_kinematic"/>
+            <child link="camera_optical_frame"/>
+            <origin xyz="0 0 0" rpy="${PI/2} ${-PI/2} 0"/>
         </joint>
-        <link name="camera_optical_frame"/>
-        <xacro:if value="${use_sim_time}">
-            <!-- this joint rotates camera because Gazebo uses YZ plane instead of XY -->
-            <joint name="camera_optical_joint" type="fixed">
-                <parent link="camera_link"/>
-                <child link="camera_optical_frame"/>
-                <origin xyz="0 0 0" rpy="${PI/2} ${-PI/2} 0"/>
-            </joint>
-        </xacro:if>
-        <xacro:unless value="${use_sim_time}">
-            <joint name="camera_optical_joint" type="fixed">
-                <parent link="camera_link"/>
-                <child link="camera_optical_frame"/>
-                <origin xyz="0 0 0.07" rpy="0 0 0"/>
-            </joint>
-        </xacro:unless>
         <gazebo reference="camera_optical_frame">
             <sensor name="rgbd_camera" type="rgbd_camera">

File: urdf/weeder_robot.xacro (robot description, xacro)
@@ -5,7 +5,5 @@
     <xacro:arg name= "is_light" default="true"/>
     <xacro:arg name= "controller_yaml" default=""/>
-    <xacro:arg name= "use_camera" default="false"/>
-    <xacro:arg name= "use_sim_time" default="true"/>
-    <xacro:macro name="weeder_robot" params="is_light use_camera controller_yaml use_sim_time">
+    <xacro:macro name="weeder_robot" params="is_light controller_yaml">
         <!-- Including base and arm xacro files -->
         <xacro:include filename="$(find arm_mazzolini)/urdf/bunker_fake.xacro"/>
@@ -23,8 +21,6 @@
             <origin xyz="0 -0.3 0.235" rpy="0 0 -${PI/2}"/>
         </joint>
-        <!-- Include depth camera if requested -->
-        <xacro:if value="${use_camera}">
-            <xacro:depth_camera is_light="${is_light}" use_sim_time="${use_sim_time}"/>
-        </xacro:if>
+        <!-- Include depth camera -->
+        <xacro:depth_camera is_light="${is_light}"/>
         <!-- Ros2 Control -->
         <ros2_control name="weeder_controller" type="system">
@@ -53,13 +49,16 @@
                 <topic>force_torque_sensor</topic>
             </sensor> -->
-            <plugin
-                filename="libignition-gazebo-pose-publisher-system.so"
-                name="ignition::gazebo::systems::PosePublisher">
+            <plugin filename="ignition-gazebo-pose-publisher-system"
+                    name="ignition::gazebo::systems::PosePublisher">
                 <publish_model_pose>true</publish_model_pose>
-                <publish_link_pose>true</publish_link_pose>
-                <update_frequency>20</update_frequency>
+                <publish_link_pose>false</publish_link_pose>
+                <publish_collision_pose>false</publish_collision_pose>
+                <publish_visual_pose>false</publish_visual_pose>
+                <publish_sensor_pose>false</publish_sensor_pose>
+                <use_pose_vector_msg>true</use_pose_vector_msg>
+                <update_frequency>50</update_frequency>
             </plugin>
         </gazebo>
     </xacro:macro>
-    <xacro:weeder_robot is_light="$(arg is_light)" use_camera="$(arg use_camera)" controller_yaml="$(arg controller_yaml)" use_sim_time="$(arg use_sim_time)"/>
+    <xacro:weeder_robot is_light="$(arg is_light)" controller_yaml="$(arg controller_yaml)"/>
 </robot>
